Commit message: some change in sim

File: car.urdf (robot description, URDF)
Before this commit: robot navgroup, 12 links, 11 joints
Joints:
- joint back_left_wheel_joint: limit velocity=0.05 -> (none)
- joint back_right_wheel_joint: limit velocity=0.05 -> (none)
- joint front_left_wheel_joint: limit velocity=0.05 -> (none)
- joint front_right_wheel_joint: limit velocity=0.05 -> (none)
